File: controller.sch (EAGLE design)
At the start: 8 parts, among them X1 PUSHBUTTON_LED

Commit message: board layout, should work
Parts:
- removed DISPLAY: C-GRID-16-70543, con-molex:C-GRID-16-70543
- removed U$2: LEVELSHIFTER, local:LEVELSHIFTER
- added C1: 47u, rcl:CPOL-EUB45181B
- added DIS1: TUXGR_16X2_R2, display-lcd:TUXGR_16X2_R2
- added Q1, Q2, Q3, Q4: BSS138, local:BSS138
- added R1, R2: 220, eagle-ltspice:R
- added R10, R11, R4, R5, R6, R7, R8, R9: 10k, eagle-ltspice:R
- added R3: 10k, pot:TRIM_EU-CA9V
- added U$4: PWR_CONV, local:PWR_CONV
Connections:
- removed net N$6: U$2G$1.LV2, U$3.SDA
- removed net N$9: ARDUINO1.D8, RELAIS.3
- new net N$17: ARDUINO1.A6, X1G$1.2, X1G$1.4, X1G$1.6
- new net N$18: DIS1.NC@1, R1.1
- new net N$19: ARDUINO1.D4, DIS1.D7
- new net SS_RFID_3V3: Q2.S, R6.1, U$3.SDA
- net +3V3: now also C1.+, Q1.G, Q2.G, Q3.G, Q4.G, R10.2, R4.2, R6.2, R8.2, U$4.VOUT; no longer U$2G$5.PWR2
- net +5V: now also DIS1.VCC, PWR-2.S, R1.2, R11.2, R3.E, R5.2, R7.2, R9.2, U$4.VIN; no longer DISPLAY-15.S, DISPLAY-2.S, U$2G$5.PWR1
- net GND: now also C1.-, DIS1.GND, DIS1.NC@2, DIS1.R/W, R2.2, R3.A, U$4.GND, X1G$1.5; no longer DISPLAY-1.S, DISPLAY-16.S, DISPLAY-5.S, U$2G$5.GND, X1G$1.2, X1G$1.4, X1G$1.6, X1G$2.C
- net MISO: now also Q4.D, R11.1; no longer U$2G$3.HV2
- net MOSI: now also Q3.D, R9.1; no longer U$2G$2.HV2
- net N$1: now also R2.1, X1G$2.C; no longer ARDUINO1.RX, X1G$2.A
- net N$10: now also ARDUINO1.D7, DIS1.D4; no longer ARDUINO1.D5, DISPLAY-11.S
- net N$11: now also ARDUINO1.A7, X1G$2.A; no longer ARDUINO1.TX, X1G$1.5
- net N$12: now also ARDUINO1.D8, DIS1.E; no longer ARDUINO1.D6, DISPLAY-6.S
- net N$13: now also ARDUINO1.D9, DIS1.RS; no longer ARDUINO1.D7, DISPLAY-4.S
- net N$14: now also ARDUINO1.D6, DIS1.D5; no longer ARDUINO1.D4, DISPLAY-12.S
- net N$15: now also RELAIS.2; no longer DISPLAY-13.S
- net N$16: now also RELAIS.3; no longer DISPLAY-14.S
- net N$2: now also Q1.S, R4.1; no longer U$2G$4.LV2
- net N$3: now also Q3.S, R8.1; no longer U$2G$2.LV2
- net N$4: now also Q4.S, R10.1; no longer U$2G$3.LV2
- net N$5: now also ARDUINO1.A0; no longer ARDUINO1.A3
- net N$7: now also ARDUINO1.D5, DIS1.D6; no longer ARDUINO1.RAW, PWR-2.S
- net N$8: now also DIS1.CONTR, R3.S; no longer ARDUINO1.D9, RELAIS.2
- net SCK: now also Q1.D, R5.1; no longer U$2G$4.HV2
- net SS_RFID: now also Q2.D, R7.1; no longer U$2G$1.HV2
Other:
- moved on the sheet: PWR-1, PWR-2, RELAIS, X1G$2
